Commit message: Cleaning up

File: wam_description/urdf/barrett_hand.urdf.xacro (robot description, xacro)
@@ -13,13 +13,15 @@
       <visual>
 	<origin rpy="1.57 0 -3.14" xyz="0.045 -0.0535 0.0148"/>
-	<geometry name="link_bhand_base_visual">
-          <mesh filename="package://wam_description/meshes/bhand_base.STL" scale="0.001 0.001 0.001" />
+	<geometry>
+          <mesh filename="package://wam_description/meshes/bhand_base.STL"
+		scale="0.001 0.001 0.001" />
 	</geometry>
 	<base_color />
       </visual>
-      <collision name="bhand_base_collision">
+      <collision>
 	<origin rpy="1.57 0 -3.14" xyz="0.045 -0.0535 0.0148"/>
-	<geometry name="link_bhand_base_collision">
-          <mesh filename="package://wam_description/meshes/bhand_base.STL" scale="0.001 0.001 0.001" />
+	<geometry>
+          <mesh filename="package://wam_description/meshes/bhand_base.STL"
+		scale="0.001 0.001 0.001" />
 	</geometry>
 	<contact_coefficients kd="1.0" kp="1000.0" mu="0"/>
@@ -34,193 +36,196 @@
       <visual>
 	<origin rpy="1.57 0 1.57" xyz="-0.0525 -0.0705 -0.025"/>
-	<geometry name="link_bhand_f11_visual">
-          <mesh filename="package://wam_description/meshes/bhand_link1.STL" scale="0.001 0.001 0.001" />
+	<geometry>
+          <mesh filename="package://wam_description/meshes/bhand_link1.STL"
+		scale="0.001 0.001 0.001" />
+	</geometry>
+	<material name="">
+          <color rgba="0.796078431372549 0.796078431372549 0.752941176470588
+		       1" />
+	</material>
+      </visual>
+      <collision>
+	<origin rpy="1.57 0 1.57" xyz="-0.0525 -0.0705 -0.025"/>
+	<geometry>
+          <mesh filename="package://wam_description/meshes/bhand_link1.STL"
+		scale="0.001 0.001 0.001" />
+	</geometry>
+	<contact_coefficients kd="1.0" kp="1000.0" mu="0"/>
+      </collision>
+    </link>
+    <link name="${prefix}link21">
+      <inertial>
+  	<mass value="0.001"/>
+	<origin xyz="0 0 0" />
+	<inertia ixx="1.0" ixy="0.0" ixz="0.0" iyy="1.0" iyz="0.0" izz="1.0"/>
+      </inertial>
+      <visual>
+	<origin rpy="1.57 0 1.57" xyz="-0.0525 -0.0705 -0.025"/>
+	<geometry>
+          <mesh filename="package://wam_description/meshes/bhand_link1.STL"
+		scale="0.001 0.001 0.001" />
 	</geometry>
 	<material
             name="">
-          <color
-              rgba="0.796078431372549 0.796078431372549 0.752941176470588 1" />
+          <color rgba="0.796078431372549 0.796078431372549 0.752941176470588
+		       1" />
 	</material>
       </visual>
       <collision>
 	<origin rpy="1.57 0 1.57" xyz="-0.0525 -0.0705 -0.025"/>
-	<geometry name="link_bhand_f11_collision">
-          <mesh filename="package://wam_description/meshes/bhand_link1.STL" scale="0.001 0.001 0.001" />
-	</geometry>
-	<contact_coefficients kd="1.0" kp="1000.0" mu="0"/>
-      </collision>
-    </link>
-    #LINK BHAND LINK F21
-    <link name="${prefix}link21">
-      <inertial>
-  	<mass value="0.001"/>
-	<origin xyz="0 0 0" />
-	<inertia ixx="1.0" ixy="0.0" ixz="0.0" iyy="1.0" iyz="0.0" izz="1.0"/>
-      </inertial>
-      <visual>
-	<origin rpy="1.57 0 1.57" xyz="-0.0525 -0.0705 -0.025"/>
-	<geometry name="link_bhand_f21_visual">
-          <mesh filename="package://wam_description/meshes/bhand_link1.STL" scale="0.001 0.001 0.001" />
+	<geometry>
+          <mesh filename="package://wam_description/meshes/bhand_link1.STL"
+		scale="0.001 0.001 0.001" />
+	</geometry>
+	<contact_coefficients kd="1.0" kp="1000.0" mu="0"/>
+      </collision>
+    </link>
+    <link name="${prefix}link12">
+      <inertial>
+  	<mass value="0.001"/>
+	<origin xyz="0 0 0" />
+	<inertia ixx="1.0" ixy="0.0" ixz="0.0" iyy="1.0" iyz="0.0" izz="1.0"/>
+      </inertial>
+      <visual>
+	<origin rpy="0 1.57 3.83972" xyz="0.0418 0.1115 0.0456"/>
+	<geometry>
+          <mesh filename="package://wam_description/meshes/bhand_link2.STL"
+		scale="0.001 0.001 0.001" />
+	</geometry>
+	<material name="">
+          <color rgba="0.796078431372549 0.796078431372549 0.752941176470588 1" />
+	</material>
+      </visual>
+      <collision>
+	<origin rpy="0 1.57 3.83972" xyz="0.0418 0.1115 0.0456"/>
+	<geometry>
+          <mesh filename="package://wam_description/meshes/bhand_link2.STL"
+		scale="0.001 0.001 0.001" />
+	</geometry>
+	<contact_coefficients kd="1.0" kp="1000.0" mu="0"/>
+      </collision>
+    </link>
+    <link name="${prefix}link22">
+      <inertial>
+  	<mass value="0.001"/>
+	<origin xyz="0 0 0" />
+	<inertia ixx="1.0" ixy="0.0" ixz="0.0" iyy="1.0" iyz="0.0" izz="1.0"/>
+      </inertial>
+      <visual>
+	<origin rpy="0 1.57 3.83972" xyz="0.0418 0.1115 0.0456"/>
+	<geometry>
+          <mesh filename="package://wam_description/meshes/bhand_link2.STL"
+		scale="0.001 0.001 0.001" />
+	</geometry>
+	<material name="">
+          <color rgba="0.796078431372549 0.796078431372549 0.752941176470588
+		       1" />
+	</material>
+      </visual>
+      <collision>
+	<origin rpy="0 1.57 3.83972" xyz="0.0418 0.1115 0.0456"/>
+	<geometry>
+          <mesh filename="package://wam_description/meshes/bhand_link2.STL"
+		scale="0.001 0.001 0.001" />
+	</geometry>
+	<contact_coefficients kd="1.0" kp="1000.0" mu="0"/>
+      </collision>
+    </link>
+    <link name="${prefix}link32">
+      <inertial>
+  	<mass value="0.001"/>
+	<origin xyz="0 0 0" />
+	<inertia ixx="1.0" ixy="0.0" ixz="0.0" iyy="1.0" iyz="0.0" izz="1.0"/>
+      </inertial>
+      <visual>
+	<origin rpy="0 1.57 3.83972" xyz="0.0418 0.1115 0.0456"/>
+	<geometry>
+          <mesh filename="package://wam_description/meshes/bhand_link2.STL"
+		scale="0.001 0.001 0.001" />
+	</geometry>
+	<material name="">
+          <color rgba="0.796078431372549 0.796078431372549 0.752941176470588
+		       1" />
+	</material>
+      </visual>
+      <collision>
+	<origin rpy="0 1.57 3.83972" xyz="0.0418 0.1115 0.0456"/>
+	<geometry>
+          <mesh filename="package://wam_description/meshes/bhand_link2.STL"
+		scale="0.001 0.001 0.001" />
+	</geometry>
+	<contact_coefficients kd="1.0" kp="1000.0" mu="0"/>
+      </collision>
+    </link>
+    <link name="${prefix}link13">
+      <inertial>
+  	<mass value="0.001"/>
+	<origin xyz="0 0 0" />
+	<inertia ixx="1.0" ixy="0.0" ixz="0.0" iyy="1.0" iyz="0.0" izz="1.0"/>
+      </inertial>
+      <visual>
+	<origin rpy="3.92699 1.57 0" xyz="0.108 0.039 0.046"/>
+	<geometry>
+          <mesh filename="package://wam_description/meshes/bhand_link3.STL"
+		scale="0.001 0.001 0.001" />
+	</geometry>
+	<material name="">
+          <color rgba="0.796078431372549 0.796078431372549 0.752941176470588
+		       1" />
+	</material>
+      </visual>
+      <collision>
+	<origin rpy="3.92699 1.57 0" xyz="0.108 0.039 0.046"/>
+	<geometry>
+          <mesh filename="package://wam_description/meshes/bhand_link3.STL"
+		scale="0.001 0.001 0.001" />
+	</geometry>
+	<contact_coefficients kd="1.0" kp="1000.0" mu="0"/>
+      </collision>
+    </link>
+    <link name="${prefix}link23">
+      <inertial>
+  	<mass value="0.001"/>
+	<origin xyz="0 0 0" />
+	<inertia ixx="1.0" ixy="0.0" ixz="0.0" iyy="1.0" iyz="0.0" izz="1.0"/>
+      </inertial>
+      <visual>
+	<origin rpy="3.92699 1.57 0" xyz="0.108 0.039 0.046"/>
+	<geometry name="link_bhand_f23_visual">
+          <mesh filename="package://wam_description/meshes/bhand_link3.STL"
+		scale="0.001 0.001 0.001" />
 	</geometry>
 	<material
             name="">
-          <color
-              rgba="0.796078431372549 0.796078431372549 0.752941176470588 1" />
-	</material>
-      </visual>
-      <collision>
-	<origin rpy="1.57 0 1.57" xyz="-0.0525 -0.0705 -0.025"/>
-	<geometry name="link_bhand_f21_collision">
-          <mesh filename="package://wam_description/meshes/bhand_link1.STL" scale="0.001 0.001 0.001" />
-	</geometry>
-	<contact_coefficients kd="1.0" kp="1000.0" mu="0"/>
-      </collision>
-    </link>
-    #LINK BHAND LINK F12
-    <link name="${prefix}link12">
-      <inertial>
-  	<mass value="0.001"/>
-	<origin xyz="0 0 0" />
-	<inertia ixx="1.0" ixy="0.0" ixz="0.0" iyy="1.0" iyz="0.0" izz="1.0"/>
-      </inertial>
-      <visual>
-	<origin rpy="0 1.57 3.83972" xyz="0.0418 0.1115 0.0456"/>
-	<geometry name="link_bhand_f12_visual">
-          <mesh filename="package://wam_description/meshes/bhand_link2.STL" scale="0.001 0.001 0.001" />
+          <color rgba="0.796078431372549 0.796078431372549 0.752941176470588
+		       1" />
+	</material>
+      </visual>
+      <collision>
+	<origin rpy="3.92699 1.57 0" xyz="0.108 0.039 0.046"/>
+	<geometry name="link_bhand_f23_collision">
+          <mesh filename="package://wam_description/meshes/bhand_link3.STL"
+		scale="0.001 0.001 0.001" />
+	</geometry>
+	<contact_coefficients kd="1.0" kp="1000.0" mu="0"/>
+      </collision>
+    </link>
+    #LINK BHAND LINK F33
+    <link name="${prefix}link33">
+      <inertial>
+  	<mass value="0.001"/>
+	<origin xyz="0 0 0" />
+	<inertia ixx="1.0" ixy="0.0" ixz="0.0" iyy="1.0" iyz="0.0" izz="1.0"/>
+      </inertial>
+      <visual>
+	<origin rpy="3.92699 1.57 0" xyz="0.108 0.039 0.046"/>
+	<geometry>
+          <mesh filename="package://wam_description/meshes/bhand_link3.STL"
+		scale="0.001 0.001 0.001" />
 	</geometry>
 	<material
             name="">
-          <color
-              rgba="0.796078431372549 0.796078431372549 0.752941176470588 1" />
-	</material>
-      </visual>
-      <collision>
-	<origin rpy="0 1.57 3.83972" xyz="0.0418 0.1115 0.0456"/>
-	<geometry name="link_bhand_f12_collision">
-          <mesh filename="package://wam_description/meshes/bhand_link2.STL" scale="0.001 0.001 0.001" />
-	</geometry>
-	<contact_coefficients kd="1.0" kp="1000.0" mu="0"/>
-      </collision>
-    </link>
-    #LINK BHAND LINK F22
-    <link name="${prefix}link22">
-      <inertial>
-  	<mass value="0.001"/>
-	<origin xyz="0 0 0" />
-	<inertia ixx="1.0" ixy="0.0" ixz="0.0" iyy="1.0" iyz="0.0" izz="1.0"/>
-      </inertial>
-      <visual>
-	<origin rpy="0 1.57 3.83972" xyz="0.0418 0.1115 0.0456"/>
-	<geometry name="link_bhand_f22_visual">
-          <mesh filename="package://wam_description/meshes/bhand_link2.STL" scale="0.001 0.001 0.001" />
-	</geometry>
-	<material
-            name="">
-          <color
-              rgba="0.796078431372549 0.796078431372549 0.752941176470588 1" />
-	</material>
-      </visual>
-      <collision>
-	<origin rpy="0 1.57 3.83972" xyz="0.0418 0.1115 0.0456"/>
-	<geometry name="link_bhand_f22_collision">
-          <mesh filename="package://wam_description/meshes/bhand_link2.STL" scale="0.001 0.001 0.001" />
-	</geometry>
-	<contact_coefficients kd="1.0" kp="1000.0" mu="0"/>
-      </collision>
-    </link>
-    #LINK BHAND LINK F32
-    <link name="${prefix}link32">
-      <inertial>
-  	<mass value="0.001"/>
-	<origin xyz="0 0 0" />
-	<inertia ixx="1.0" ixy="0.0" ixz="0.0" iyy="1.0" iyz="0.0" izz="1.0"/>
-      </inertial>
-      <visual>
-	<origin rpy="0 1.57 3.83972" xyz="0.0418 0.1115 0.0456"/>
-	<geometry name="link_bhand_f32_visual">
-          <mesh filename="package://wam_description/meshes/bhand_link2.STL" scale="0.001 0.001 0.001" />
-	</geometry>
-	<material
-            name="">
-          <color
-              rgba="0.796078431372549 0.796078431372549 0.752941176470588 1" />
-	</material>
-      </visual>
-      <collision>
-	<origin rpy="0 1.57 3.83972" xyz="0.0418 0.1115 0.0456"/>
-	<geometry name="link_bhand_f32_collision">
-          <mesh filename="package://wam_description/meshes/bhand_link2.STL" scale="0.001 0.001 0.001" />
-	</geometry>
-	<contact_coefficients kd="1.0" kp="1000.0" mu="0"/>
-      </collision>
-    </link>
-    #LINK BHAND LINK F13
-    <link name="${prefix}link13">
-      <inertial>
-  	<mass value="0.001"/>
-	<origin xyz="0 0 0" />
-	<inertia ixx="1.0" ixy="0.0" ixz="0.0" iyy="1.0" iyz="0.0" izz="1.0"/>
-      </inertial>
-      <visual>
-	<origin rpy="3.92699 1.57 0" xyz="0.108 0.039 0.046"/>
-	<geometry name="link_bhand_f13_visual">
-          <mesh filename="package://wam_description/meshes/bhand_link3.STL" scale="0.001 0.001 0.001" />
-	</geometry>
-	<material
-            name="">
-          <color
-              rgba="0.796078431372549 0.796078431372549 0.752941176470588 1" />
-	</material>
-      </visual>
-      <collision>
-	<origin rpy="3.92699 1.57 0" xyz="0.108 0.039 0.046"/>
-	<geometry name="link_bhand_f13_collision">
-          <mesh filename="package://wam_description/meshes/bhand_link3.STL" scale="0.001 0.001 0.001" />
-	</geometry>
-	<contact_coefficients kd="1.0" kp="1000.0" mu="0"/>
-      </collision>
-    </link>
-    #LINK BHAND LINK F23
-    <link name="${prefix}link23">
-      <inertial>
-  	<mass value="0.001"/>
-	<origin xyz="0 0 0" />
-	<inertia ixx="1.0" ixy="0.0" ixz="0.0" iyy="1.0" iyz="0.0" izz="1.0"/>
-      </inertial>
-      <visual>
-	<origin rpy="3.92699 1.57 0" xyz="0.108 0.039 0.046"/>
-	<geometry name="link_bhand_f23_visual">
-          <mesh filename="package://wam_description/meshes/bhand_link3.STL" scale="0.001 0.001 0.001" />
-	</geometry>
-	<material
-            name="">
-          <color
-              rgba="0.796078431372549 0.796078431372549 0.752941176470588 1" />
-	</material>
-      </visual>
-      <collision>
-	<origin rpy="3.92699 1.57 0" xyz="0.108 0.039 0.046"/>
-	<geometry name="link_bhand_f23_collision">
-          <mesh filename="package://wam_description/meshes/bhand_link3.STL" scale="0.001 0.001 0.001" />
-	</geometry>
-	<contact_coefficients kd="1.0" kp="1000.0" mu="0"/>
-      </collision>
-    </link>
-    #LINK BHAND LINK F33
-    <link name="${prefix}link33">
-      <inertial>
-  	<mass value="0.001"/>
-	<origin xyz="0 0 0" />
-	<inertia ixx="1.0" ixy="0.0" ixz="0.0" iyy="1.0" iyz="0.0" izz="1.0"/>
-      </inertial>
-      <visual>
-	<origin rpy="3.92699 1.57 0" xyz="0.108 0.039 0.046"/>
-	<geometry name="link_bhand_f33_visual">
-          <mesh filename="package://wam_description/meshes/bhand_link3.STL" scale="0.001 0.001 0.001" />
-	</geometry>
-	<material
-            name="">
-          <color
-              rgba="0.796078431372549 0.796078431372549 0.752941176470588 1" />
+          <color rgba="0.796078431372549 0.796078431372549 0.752941176470588
+		       1" />
 	</material>
       </visual>
@@ -228,5 +233,6 @@
 	<origin rpy="3.92699 1.57 0" xyz="0.108 0.039 0.046"/>
 	<geometry name="link_bhand_f33_collision">
-          <mesh filename="package://wam_description/meshes/bhand_link3.STL" scale="0.001 0.001 0.001" />
+          <mesh filename="package://wam_description/meshes/bhand_link3.STL"
+		scale="0.001 0.001 0.001" />
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