Commit message: Cleanup Barrett hand URDF

File: wam_description/urdf/barrett_hand.urdf.xacro (robot description, xacro)
@@ -2,241 +2,11 @@
 <robot xmlns:xacro="http://www.ros.org/wiki/xacro"
        xmlns:controller="http://playerstage.sourceforge.net/gazebo/xmlschema/#controller">
-  <include filename="$(find wam_description
-		     )/urdf/palm_tactile_sensors.urdf.xacro" />
   <xacro:macro name="barrett_hand" params="prefix parent_link *origin">
-    <link name="${prefix}base">
-      <inertial>
-  	<mass value="0.001"/>
-	<origin xyz="0 0 0" />
-	<inertia ixx="1.0" ixy="0.0" ixz="0.0" iyy="1.0" iyz="0.0" izz="1.0"/>
-      </inertial>
-      <visual>
-	<origin rpy="1.57 0 -3.14" xyz="0.045 -0.0535 0.0148"/>
-	<geometry>
-          <mesh filename="package://wam_description/meshes/bhand_base.STL"
-		scale="0.001 0.001 0.001" />
-	</geometry>
-	<base_color />
-      </visual>
-      <collision>
-	<origin rpy="1.57 0 -3.14" xyz="0.045 -0.0535 0.0148"/>
-	<geometry>
-          <mesh filename="package://wam_description/meshes/bhand_base.STL"
-		scale="0.001 0.001 0.001" />
-	</geometry>
-	<contact_coefficients kd="1.0" kp="1000.0" mu="0"/>
-      </collision>
-    </link>
-    <link name="${prefix}link11">
-      <inertial>
-  	<mass value="0.001"/>
-	<origin xyz="0 0 0" />
-	<inertia ixx="1.0" ixy="0.0" ixz="0.0" iyy="1.0" iyz="0.0" izz="1.0"/>
-      </inertial>
-      <visual>
-	<origin rpy="1.57 0 1.57" xyz="-0.0525 -0.0705 -0.025"/>
-	<geometry>
-          <mesh filename="package://wam_description/meshes/bhand_link1.STL"
-		scale="0.001 0.001 0.001" />
-	</geometry>
-	<material name="">
-          <color rgba="0.796078431372549 0.796078431372549 0.752941176470588
-		       1" />
-	</material>
-      </visual>
-      <collision>
-	<origin rpy="1.57 0 1.57" xyz="-0.0525 -0.0705 -0.025"/>
-	<geometry>
-          <mesh filename="package://wam_description/meshes/bhand_link1.STL"
-		scale="0.001 0.001 0.001" />
-	</geometry>
-	<contact_coefficients kd="1.0" kp="1000.0" mu="0"/>
-      </collision>
-    </link>
-    <link name="${prefix}link21">
-      <inertial>
-  	<mass value="0.001"/>
-	<origin xyz="0 0 0" />
-	<inertia ixx="1.0" ixy="0.0" ixz="0.0" iyy="1.0" iyz="0.0" izz="1.0"/>
-      </inertial>
-      <visual>
-	<origin rpy="1.57 0 1.57" xyz="-0.0525 -0.0705 -0.025"/>
-	<geometry>
-          <mesh filename="package://wam_description/meshes/bhand_link1.STL"
-		scale="0.001 0.001 0.001" />
-	</geometry>
-	<material
-            name="">
-          <color rgba="0.796078431372549 0.796078431372549 0.752941176470588
-		       1" />
-	</material>
-      </visual>
-      <collision>
-	<origin rpy="1.57 0 1.57" xyz="-0.0525 -0.0705 -0.025"/>
-	<geometry>
-          <mesh filename="package://wam_description/meshes/bhand_link1.STL"
-		scale="0.001 0.001 0.001" />
-	</geometry>
-	<contact_coefficients kd="1.0" kp="1000.0" mu="0"/>
-      </collision>
-    </link>
-    <link name="${prefix}link12">
-      <inertial>
-  	<mass value="0.001"/>
-	<origin xyz="0 0 0" />
-	<inertia ixx="1.0" ixy="0.0" ixz="0.0" iyy="1.0" iyz="0.0" izz="1.0"/>
-      </inertial>
-      <visual>
-	<origin rpy="0 1.57 3.83972" xyz="0.0418 0.1115 0.0456"/>
-	<geometry>
-          <mesh filename="package://wam_description/meshes/bhand_link2.STL"
-		scale="0.001 0.001 0.001" />
-	</geometry>
-	<material name="">
-          <color rgba="0.796078431372549 0.796078431372549 0.752941176470588 1" />
-	</material>
-      </visual>
-      <collision>
-	<origin rpy="0 1.57 3.83972" xyz="0.0418 0.1115 0.0456"/>
-	<geometry>
-          <mesh filename="package://wam_description/meshes/bhand_link2.STL"
-		scale="0.001 0.001 0.001" />
-	</geometry>
-	<contact_coefficients kd="1.0" kp="1000.0" mu="0"/>
-      </collision>
-    </link>
-    <link name="${prefix}link22">
-      <inertial>
-  	<mass value="0.001"/>
-	<origin xyz="0 0 0" />
-	<inertia ixx="1.0" ixy="0.0" ixz="0.0" iyy="1.0" iyz="0.0" izz="1.0"/>
-      </inertial>
-      <visual>
-	<origin rpy="0 1.57 3.83972" xyz="0.0418 0.1115 0.0456"/>
-	<geometry>
-          <mesh filename="package://wam_description/meshes/bhand_link2.STL"
-		scale="0.001 0.001 0.001" />
-	</geometry>
-	<material name="">
-          <color rgba="0.796078431372549 0.796078431372549 0.752941176470588
-		       1" />
-	</material>
-      </visual>
-      <collision>
-	<origin rpy="0 1.57 3.83972" xyz="0.0418 0.1115 0.0456"/>
-	<geometry>
-          <mesh filename="package://wam_description/meshes/bhand_link2.STL"
-		scale="0.001 0.001 0.001" />
-	</geometry>
-	<contact_coefficients kd="1.0" kp="1000.0" mu="0"/>
-      </collision>
-    </link>
-    <link name="${prefix}link32">
-      <inertial>
-  	<mass value="0.001"/>
-	<origin xyz="0 0 0" />
-	<inertia ixx="1.0" ixy="0.0" ixz="0.0" iyy="1.0" iyz="0.0" izz="1.0"/>
-      </inertial>
-      <visual>
-	<origin rpy="0 1.57 3.83972" xyz="0.0418 0.1115 0.0456"/>
-	<geometry>
-          <mesh filename="package://wam_description/meshes/bhand_link2.STL"
-		scale="0.001 0.001 0.001" />
-	</geometry>
-	<material name="">
-          <color rgba="0.796078431372549 0.796078431372549 0.752941176470588
-		       1" />
-	</material>
-      </visual>
-      <collision>
-	<origin rpy="0 1.57 3.83972" xyz="0.0418 0.1115 0.0456"/>
-	<geometry>
-          <mesh filename="package://wam_description/meshes/bhand_link2.STL"
-		scale="0.001 0.001 0.001" />
-	</geometry>
-	<contact_coefficients kd="1.0" kp="1000.0" mu="0"/>
-      </collision>
-    </link>
-    <link name="${prefix}link13">
-      <inertial>
-  	<mass value="0.001"/>
-	<origin xyz="0 0 0" />
-	<inertia ixx="1.0" ixy="0.0" ixz="0.0" iyy="1.0" iyz="0.0" izz="1.0"/>
-      </inertial>
-      <visual>
-	<origin rpy="3.92699 1.57 0" xyz="0.108 0.039 0.046"/>
-	<geometry>
-          <mesh filename="package://wam_description/meshes/bhand_link3.STL"
-		scale="0.001 0.001 0.001" />
-	</geometry>
-	<material name="">
-          <color rgba="0.796078431372549 0.796078431372549 0.752941176470588
-		       1" />
-	</material>
-      </visual>
-      <collision>
-	<origin rpy="3.92699 1.57 0" xyz="0.108 0.039 0.046"/>
-	<geometry>
-          <mesh filename="package://wam_description/meshes/bhand_link3.STL"
-		scale="0.001 0.001 0.001" />
-	</geometry>
-	<contact_coefficients kd="1.0" kp="1000.0" mu="0"/>
-      </collision>
-    </link>
-    <link name="${prefix}link23">
-      <inertial>
-  	<mass value="0.001"/>
-	<origin xyz="0 0 0" />
-	<inertia ixx="1.0" ixy="0.0" ixz="0.0" iyy="1.0" iyz="0.0" izz="1.0"/>
-      </inertial>
-      <visual>
-	<origin rpy="3.92699 1.57 0" xyz="0.108 0.039 0.046"/>
-	<geometry name="link_bhand_f23_visual">
-          <mesh filename="package://wam_description/meshes/bhand_link3.STL"
-		scale="0.001 0.001 0.001" />
-	</geometry>
-	<material
-            name="">
-          <color rgba="0.796078431372549 0.796078431372549 0.752941176470588
-		       1" />
-	</material>
-      </visual>
-      <collision>
-	<origin rpy="3.92699 1.57 0" xyz="0.108 0.039 0.046"/>
-	<geometry name="link_bhand_f23_collision">
-          <mesh filename="package://wam_description/meshes/bhand_link3.STL"
-		scale="0.001 0.001 0.001" />
-	</geometry>
-	<contact_coefficients kd="1.0" kp="1000.0" mu="0"/>
-      </collision>
-    </link>
-    #LINK BHAND LINK F33
-    <link name="${prefix}link33">
-      <inertial>
-  	<mass value="0.001"/>
-	<origin xyz="0 0 0" />
-	<inertia ixx="1.0" ixy="0.0" ixz="0.0" iyy="1.0" iyz="0.0" izz="1.0"/>
-      </inertial>
-      <visual>
-	<origin rpy="3.92699 1.57 0" xyz="0.108 0.039 0.046"/>
-	<geometry>
-          <mesh filename="package://wam_description/meshes/bhand_link3.STL"
-		scale="0.001 0.001 0.001" />
-	</geometry>
-	<material
-            name="">
-          <color rgba="0.796078431372549 0.796078431372549 0.752941176470588
-		       1" />
-	</material>
-      </visual>
-      <collision>
-	<origin rpy="3.92699 1.57 0" xyz="0.108 0.039 0.046"/>
-	<geometry name="link_bhand_f33_collision">
-          <mesh filename="package://wam_description/meshes/bhand_link3.STL"
-		scale="0.001 0.001 0.001" />
-	</geometry>
-	<contact_coefficients kd="1.0" kp="1000.0" mu="0"/>
-      </collision>
-    </link>
+    <xacro:macro name="gray_color">
+      <material name="">
+	<color rgba="0.796078431372549 0.796078431372549 0.752941176470588 1"/>
+      </material>
+    </xacro:macro>
+    <!-- Base -->
     <joint name="${prefix}base_joint" type="fixed">
       <parent link="${parent_link}"/>
@@ -244,4 +14,28 @@
       <xacro:insert_block name="origin"/>
     </joint>
+    <link name="${prefix}base">
+      <inertial>
+  	<mass value="0.001"/>
+	<origin xyz="0 0 0" />
+	<inertia ixx="1.0" ixy="0.0" ixz="0.0" iyy="1.0" iyz="0.0" izz="1.0"/>
+      </inertial>
+      <visual>
+	<origin rpy="1.57 0 -3.14" xyz="0.045 -0.0535 0.0148"/>
+	<geometry>
+          <mesh filename="package://wam_description/meshes/bhand_base.STL"
+		scale="0.001 0.001 0.001" />
+	</geometry>
+	<xacro:gray_color/>
+      </visual>
+      <collision>
+	<origin rpy="1.57 0 -3.14" xyz="0.045 -0.0535 0.0148"/>
+	<geometry>
+          <mesh filename="package://wam_description/meshes/bhand_base.STL"
+		scale="0.001 0.001 0.001" />
+	</geometry>
+	<contact_coefficients kd="1.0" kp="1000.0" mu="0"/>
+      </collision>
+    </link>
+    <!-- Finger 1 -->
     <joint name="${prefix}j11_joint" type="revolute">
       <origin xyz="-0.02475 0.0 0.0395" rpy="0.0 0 -1.57079633" />
@@ -253,4 +47,93 @@
       <dynamics damping="1000"/>
     </joint>
+    <link name="${prefix}link11">
+      <inertial>
+  	<mass value="0.001"/>
+	<origin xyz="0 0 0" />
+	<inertia ixx="1.0" ixy="0.0" ixz="0.0" iyy="1.0" iyz="0.0" izz="1.0"/>
+      </inertial>
+      <visual>
+	<origin rpy="1.57 0 1.57" xyz="-0.0525 -0.0705 -0.025"/>
+	<geometry>
+          <mesh filename="package://wam_description/meshes/bhand_link1.STL"
+		scale="0.001 0.001 0.001" />
+	</geometry>
+	<xacro:gray_color/>
+      </visual>
+      <collision>
+	<origin rpy="1.57 0 1.57" xyz="-0.0525 -0.0705 -0.025"/>
+	<geometry>
+          <mesh filename="package://wam_description/meshes/bhand_link1.STL"
+		scale="0.001 0.001 0.001" />
+	</geometry>
+	<contact_coefficients kd="1.0" kp="1000.0" mu="0"/>
+      </collision>
+    </link>
+    <joint name="${prefix}j12_joint" type="revolute">
+      <origin xyz="0.050 0.0 0.038" rpy="1.57079633 0 0.0" />
+      <parent link="${prefix}link11"/>
+      <child link="${prefix}link12" />
+      <axis xyz="0 0 1"/>
+      <limit effort="30" velocity="1.5" lower="0.0" upper="2.44346095" />
+      <joint_properties damping="100.0" friction="1000.0" />
+      <dynamics damping="1000"/>
+    </joint >
+    <link name="${prefix}link12">
+      <inertial>
+  	<mass value="0.001"/>
+	<origin xyz="0 0 0" />
+	<inertia ixx="1.0" ixy="0.0" ixz="0.0" iyy="1.0" iyz="0.0" izz="1.0"/>
+      </inertial>
+      <visual>
+	<origin rpy="0 1.57 3.83972" xyz="0.0418 0.1115 0.0456"/>
+	<geometry>
+          <mesh filename="package://wam_description/meshes/bhand_link2.STL"
+		scale="0.001 0.001 0.001" />
+	</geometry>
+	<xacro:gray_color/>
+      </visual>
+      <collision>
+	<origin rpy="0 1.57 3.83972" xyz="0.0418 0.1115 0.0456"/>
+	<geometry>
+          <mesh filename="package://wam_description/meshes/bhand_link2.STL"
+		scale="0.001 0.001 0.001" />
+	</geometry>
+	<contact_coefficients kd="1.0" kp="1000.0" mu="0"/>
+      </collision>
+    </link>
+    <joint name="${prefix}j13_joint" type="revolute">
+      <origin xyz="0.070 0.0 0.0" rpy="0.0 0 0.0" />
+      <parent link="${prefix}link12"/>
+      <child link="${prefix}link13" />
+      <axis xyz="0 0 1"/>
+      <limit effort="30" velocity="1.5"
+	     lower="0.698131701" upper="2.44346095" />
+      <joint_properties damping="100.0" friction="1000.0" />
+      <dynamics damping="1000"/>
+    </joint >
+    <link name="${prefix}link13">
+      <inertial>
+  	<mass value="0.001"/>
+	<origin xyz="0 0 0" />
+	<inertia ixx="1.0" ixy="0.0" ixz="0.0" iyy="1.0" iyz="0.0" izz="1.0"/>
+      </inertial>
+      <visual>
+	<origin rpy="3.92699 1.57 0" xyz="0.108 0.039 0.046"/>
+	<geometry>
+          <mesh filename="package://wam_description/meshes/bhand_link3.STL"
+		scale="0.001 0.001 0.001" />
+	</geometry>
+	<xacro:gray_color/>
+      </visual>
+      <collision>
+	<origin rpy="3.92699 1.57 0" xyz="0.108 0.039 0.046"/>
+	<geometry>
+          <mesh filename="package://wam_description/meshes/bhand_link3.STL"
+		scale="0.001 0.001 0.001" />
+	</geometry>
+	<contact_coefficients kd="1.0" kp="1000.0" mu="0"/>
+      </collision>
+    </link>
+    <!-- Finger 2 -->
     <joint name="${prefix}j21_joint" type="revolute">
       <origin xyz="0.02475 0.0 0.0395" rpy="0.0 0.0 -1.57079633" />
@@ -262,13 +145,27 @@
       <dynamics damping="1000"/>
     </joint >
-    <joint name="${prefix}j12_joint" type="revolute">
-      <origin xyz="0.050 0.0 0.038" rpy="1.57079633 0 0.0" />
-      <parent link="${prefix}link11"/>
-      <child link="${prefix}link12" />
-      <axis xyz="0 0 1"/>
-      <limit effort="30" velocity="1.5" lower="0.0" upper="2.44346095" />
-      <joint_properties damping="100.0" friction="1000.0" />
-      <dynamics damping="1000"/>
-    </joint >
+    <link name="${prefix}link21">
+      <inertial>
+  	<mass value="0.001"/>
+	<origin xyz="0 0 0" />
+	<inertia ixx="1.0" ixy="0.0" ixz="0.0" iyy="1.0" iyz="0.0" izz="1.0"/>
+      </inertial>
+      <visual>
+	<origin rpy="1.57 0 1.57" xyz="-0.0525 -0.0705 -0.025"/>
+	<geometry>
+          <mesh filename="package://wam_description/meshes/bhand_link1.STL"
+		scale="0.001 0.001 0.001" />
+	</geometry>
+	<xacro:gray_color/>
+      </visual>
+      <collision>
+	<origin rpy="1.57 0 1.57" xyz="-0.0525 -0.0705 -0.025"/>
+	<geometry>
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