Commit message: Replace prefix with device_name

File: aist_barrett/urdf/barrett_hand.urdf.xacro (robot description, xacro)
@@ -2,5 +2,5 @@
 <robot xmlns:xacro="http://www.ros.org/wiki/xacro"
        xmlns:controller="http://playerstage.sourceforge.net/gazebo/xmlschema/#controller">
-  <xacro:macro name="barrett_hand" params="prefix parent_link *origin">
+  <xacro:macro name="barrett_hand" params="name parent_link *origin">
     <xacro:macro name="gray_color">
       <material name="">
@@ -9,10 +9,10 @@
     </xacro:macro>
     <!-- Base -->
-    <joint name="${prefix}base_joint" type="fixed">
+    <joint name="${name}_base_joint" type="fixed">
       <parent link="${parent_link}"/>
-      <child link="${prefix}base" />
+      <child link="${name}_base" />
       <xacro:insert_block name="origin"/>
     </joint>
-    <link name="${prefix}base">
+    <link name="${name}_base">
       <inertial>
   	<mass value="0.001"/>
@@ -38,8 +38,8 @@
     </link>
     <!-- Finger 1 -->
-    <joint name="${prefix}j11_joint" type="revolute">
+    <joint name="${name}_j11_joint" type="revolute">
       <origin xyz="-0.02475 0.0 0.0395" rpy="0.0 0 -1.57079633" />
-      <parent link="${prefix}base"/>
-      <child link="${prefix}link11" />
+      <parent link="${name}_base"/>
+      <child link="${name}_link11" />
       <axis xyz="0 0 -1"/>
       <limit effort="30" velocity="1.5" lower="0.0" upper="3.14159265" />
@@ -47,5 +47,5 @@
       <dynamics damping="1000"/>
     </joint>
-    <link name="${prefix}link11">
+    <link name="${name}_link11">
       <inertial>
   	<mass value="0.001"/>
@@ -70,8 +70,8 @@
       </collision>
     </link>
-    <joint name="${prefix}j12_joint" type="revolute">
+    <joint name="${name}_j12_joint" type="revolute">
       <origin xyz="0.050 0.0 0.038" rpy="1.57079633 0 0.0" />
-      <parent link="${prefix}link11"/>
-      <child link="${prefix}link12" />
+      <parent link="${name}_link11"/>
+      <child link="${name}_link12" />
       <axis xyz="0 0 1"/>
       <limit effort="30" velocity="1.5" lower="0.0" upper="2.44346095" />
@@ -79,31 +79,31 @@
       <dynamics damping="1000"/>
     </joint >
-    <link name="${prefix}link12">
-      <inertial>
-  	<mass value="0.001"/>
-	<origin xyz="0 0 0" />
-	<inertia ixx="1.0" ixy="0.0" ixz="0.0" iyy="1.0" iyz="0.0" izz="1.0"/>
-      </inertial>
-      <visual>
-	<origin rpy="0 1.57 3.83972" xyz="0.0418 0.1115 0.0456"/>
-	<geometry>
-          <mesh filename="package://aist_barrett/meshes/bhand_link2.STL"
-		scale="0.001 0.001 0.001" />
-	</geometry>
-	<xacro:gray_color/>
-      </visual>
-      <collision>
-	<origin rpy="0 1.57 3.83972" xyz="0.0418 0.1115 0.0456"/>
-	<geometry>
-          <mesh filename="package://aist_barrett/meshes/bhand_link2.STL"
-		scale="0.001 0.001 0.001" />
-	</geometry>
-	<contact_coefficients kd="1.0" kp="1000.0" mu="0"/>
-      </collision>
-    </link>
-    <joint name="${prefix}j13_joint" type="revolute">
+    <link name="${name}_link12">
+      <inertial>
+  	<mass value="0.001"/>
+	<origin xyz="0 0 0" />
+	<inertia ixx="1.0" ixy="0.0" ixz="0.0" iyy="1.0" iyz="0.0" izz="1.0"/>
+      </inertial>
+      <visual>
+	<origin rpy="0 1.57 3.83972" xyz="0.0418 0.1115 0.0456"/>
+	<geometry>
+          <mesh filename="package://aist_barrett/meshes/bhand_link2.STL"
+		scale="0.001 0.001 0.001" />
+	</geometry>
+	<xacro:gray_color/>
+      </visual>
+      <collision>
+	<origin rpy="0 1.57 3.83972" xyz="0.0418 0.1115 0.0456"/>
+	<geometry>
+          <mesh filename="package://aist_barrett/meshes/bhand_link2.STL"
+		scale="0.001 0.001 0.001" />
+	</geometry>
+	<contact_coefficients kd="1.0" kp="1000.0" mu="0"/>
+      </collision>
+    </link>
+    <joint name="${name}_j13_joint" type="revolute">
       <origin xyz="0.070 0.0 0.0" rpy="0.0 0 0.0" />
-      <parent link="${prefix}link12"/>
-      <child link="${prefix}link13" />
+      <parent link="${name}_link12"/>
+      <child link="${name}_link13" />
       <axis xyz="0 0 1"/>
       <limit effort="30" velocity="1.5"
@@ -112,5 +112,5 @@
       <dynamics damping="1000"/>
     </joint >
-    <link name="${prefix}link13">
+    <link name="${name}_link13">
       <inertial>
   	<mass value="0.001"/>
@@ -136,8 +136,8 @@
     </link>
     <!-- Finger 2 -->
-    <joint name="${prefix}j21_joint" type="revolute">
+    <joint name="${name}_j21_joint" type="revolute">
       <origin xyz="0.02475 0.0 0.0395" rpy="0.0 0.0 -1.57079633" />
-      <parent link="${prefix}base"/>
-      <child link="${prefix}link21" />
+      <parent link="${name}_base"/>
+      <child link="${name}_link21" />
       <axis xyz="0 0 -1"/>
       <limit effort="30" velocity="1.5" lower="-3.14159265" upper="0.0" />
@@ -145,5 +145,5 @@
       <dynamics damping="1000"/>
     </joint >
-    <link name="${prefix}link21">
+    <link name="${name}_link21">
       <inertial>
   	<mass value="0.001"/>
@@ -168,8 +168,8 @@
       </collision>
     </link>
-    <joint name="${prefix}j22_joint" type="revolute">
+    <joint name="${name}_j22_joint" type="revolute">
       <origin xyz="0.050 0.0 0.038" rpy="1.57079633 0 0.0" />
-      <parent link="${prefix}link21"/>
-      <child link="${prefix}link22" />
+      <parent link="${name}_link21"/>
+      <child link="${name}_link22" />
       <axis xyz="0 0 1"/>
       <limit effort="30" velocity="1.5" lower="0.0" upper="2.44346095" />
@@ -177,31 +177,31 @@
       <dynamics damping="1000"/>
     </joint >
-    <link name="${prefix}link22">
-      <inertial>
-  	<mass value="0.001"/>
-	<origin xyz="0 0 0" />
-	<inertia ixx="1.0" ixy="0.0" ixz="0.0" iyy="1.0" iyz="0.0" izz="1.0"/>
-      </inertial>
-      <visual>
-	<origin rpy="0 1.57 3.83972" xyz="0.0418 0.1115 0.0456"/>
-	<geometry>
-          <mesh filename="package://aist_barrett/meshes/bhand_link2.STL"
-		scale="0.001 0.001 0.001" />
-	</geometry>
-	<xacro:gray_color/>
-      </visual>
-      <collision>
-	<origin rpy="0 1.57 3.83972" xyz="0.0418 0.1115 0.0456"/>
-	<geometry>
-          <mesh filename="package://aist_barrett/meshes/bhand_link2.STL"
-		scale="0.001 0.001 0.001" />
-	</geometry>
-	<contact_coefficients kd="1.0" kp="1000.0" mu="0"/>
-      </collision>
-    </link>
-    <joint name="${prefix}j23_joint" type="revolute">
+    <link name="${name}_link22">
+      <inertial>
+  	<mass value="0.001"/>
+	<origin xyz="0 0 0" />
+	<inertia ixx="1.0" ixy="0.0" ixz="0.0" iyy="1.0" iyz="0.0" izz="1.0"/>
+      </inertial>
+      <visual>
+	<origin rpy="0 1.57 3.83972" xyz="0.0418 0.1115 0.0456"/>
+	<geometry>
+          <mesh filename="package://aist_barrett/meshes/bhand_link2.STL"
+		scale="0.001 0.001 0.001" />
+	</geometry>
+	<xacro:gray_color/>
+      </visual>
+      <collision>
+	<origin rpy="0 1.57 3.83972" xyz="0.0418 0.1115 0.0456"/>
+	<geometry>
+          <mesh filename="package://aist_barrett/meshes/bhand_link2.STL"
+		scale="0.001 0.001 0.001" />
+	</geometry>
+	<contact_coefficients kd="1.0" kp="1000.0" mu="0"/>
+      </collision>
+    </link>
+    <joint name="${name}_j23_joint" type="revolute">
       <origin xyz="0.070 0.0 0.0" rpy="0.0 0 0.0" />
-      <parent link="${prefix}link22"/>
-      <child link="${prefix}link23" />
+      <parent link="${name}_link22"/>
+      <child link="${name}_link23" />
       <axis xyz="0 0 1"/>
       <limit effort="30" velocity="1.5"
@@ -210,5 +210,5 @@
       <dynamics damping="1000"/>
     </joint >
-    <link name="${prefix}link23">
+    <link name="${name}_link23">
       <inertial>
   	<mass value="0.001"/>
@@ -234,8 +234,8 @@
     </link>
     <!-- Finger 3 -->
-    <joint name="${prefix}j32_joint" type="revolute">
+    <joint name="${name}_j32_joint" type="revolute">
       <origin xyz="0.0 0.050 0.0775" rpy="1.57079633 0 1.57079633" />
-      <parent link="${prefix}base"/>
-      <child link="${prefix}link32" />
+      <parent link="${name}_base"/>
+      <child link="${name}_link32" />
       <axis xyz="0 0 1"/>
       <limit effort="30" velocity="1.5" lower="0.0" upper="2.44346095" />
@@ -243,31 +243,31 @@
       <dynamics damping="1000"/>
     </joint >
-    <link name="${prefix}link32">
-      <inertial>
-  	<mass value="0.001"/>
-	<origin xyz="0 0 0" />
-	<inertia ixx="1.0" ixy="0.0" ixz="0.0" iyy="1.0" iyz="0.0" izz="1.0"/>
-      </inertial>
-      <visual>
-	<origin rpy="0 1.57 3.83972" xyz="0.0418 0.1115 0.0456"/>
-	<geometry>
-          <mesh filename="package://aist_barrett/meshes/bhand_link2.STL"
-		scale="0.001 0.001 0.001" />
-	</geometry>
-	<xacro:gray_color/>
-      </visual>
-      <collision>
-	<origin rpy="0 1.57 3.83972" xyz="0.0418 0.1115 0.0456"/>
-	<geometry>
-          <mesh filename="package://aist_barrett/meshes/bhand_link2.STL"
-		scale="0.001 0.001 0.001" />
-	</geometry>
-	<contact_coefficients kd="1.0" kp="1000.0" mu="0"/>
-      </collision>
-    </link>
-    <joint name="${prefix}j33_joint" type="revolute">
+    <link name="${name}_link32">
+      <inertial>
+  	<mass value="0.001"/>
+	<origin xyz="0 0 0" />
+	<inertia ixx="1.0" ixy="0.0" ixz="0.0" iyy="1.0" iyz="0.0" izz="1.0"/>
+      </inertial>
+      <visual>
+	<origin rpy="0 1.57 3.83972" xyz="0.0418 0.1115 0.0456"/>
+	<geometry>
+          <mesh filename="package://aist_barrett/meshes/bhand_link2.STL"
+		scale="0.001 0.001 0.001" />
+	</geometry>
+	<xacro:gray_color/>
+      </visual>
+      <collision>
+	<origin rpy="0 1.57 3.83972" xyz="0.0418 0.1115 0.0456"/>
+	<geometry>
+          <mesh filename="package://aist_barrett/meshes/bhand_link2.STL"
+		scale="0.001 0.001 0.001" />
+	</geometry>
+	<contact_coefficients kd="1.0" kp="1000.0" mu="0"/>
+      </collision>
+    </link>
+    <joint name="${name}_j33_joint" type="revolute">
       <origin xyz="0.070 0.0 0.0" rpy="0.0 0 0.0" />
-      <parent link="${prefix}link32"/>
-      <child link="${prefix}link33" />
+      <parent link="${name}_link32"/>
+      <child link="${name}_link33" />
       <axis xyz="0 0 1"/>
       <limit effort="30" velocity="1.5"
@@ -276,5 +276,5 @@
       <dynamics damping="1000"/>
     </joint >
-    <link name="${prefix}link33">
+    <link name="${name}_link33">
       <inertial>
   	<mass value="0.001"/>
