Commit message: WIP

File: aist_barrett/urdf/barrett_hand.urdf.xacro (robot description, xacro)
@@ -9,11 +9,12 @@
       </material>
     </xacro:macro>
-    <xacro:property name="base_height"	value="0.025"/>
-    <xacro:property name="palm_height"	value="0.061"/>
-    <xacro:property name="tip_height"	value="0.156"/>
-    <xacro:property name="half_tread"	value="0.025"/>
-    <xacro:property name="inner_x"	value="0.050"/>
-    <xacro:property name="inner_y"	value="0.000"/>
-    <xacro:property name="inner_z"	value="0.035"/>
+    <xacro:property name="base_height"		value="0.025"/>
+    <xacro:property name="palm_height"		value="0.061"/>
+    <xacro:property name="tip_height"		value="0.156"/>
+    <xacro:property name="half_tread"		value="0.025"/>
+    <xacro:property name="inner_x"		value="0.050"/>
+    <xacro:property name="inner_z"		value="0.035"/>
+    <xacro:property name="inner_finger_length"	value="0.070"/>
+    <xacro:property name="outer_finger_length"	value="0.058"/>
     <xacro:macro name="set_frame" params="name parent *origin">
       <joint name="${name}_joint" type="fixed">
@@ -64,5 +65,6 @@
       <joint name="${fingerprefix}outer_joint"
 	     type="revolute">
-	<origin xyz="0.070 0.0 0.0" rpy="0.0 0.0 ${radians(35)}"/>
+	<origin xyz="${inner_finger_length} 0.0 0.0"
+		rpy="0.0 0.0 ${radians(35)}"/>
 	<parent link="${fingerprefix}inner_link"/>
 	<child  link="${fingerprefix}outer_link"/>
@@ -105,5 +107,5 @@
       <xacro:set_frame name="${fingerprefix}tip_link"
 		       parent="${fingerprefix}outer_link">
-	<origin xyz="0.058 0 0" rpy="0 ${radians(-90)} 0"/>
+	<origin xyz="${outer_finger_length} 0 0" rpy="0 ${radians(-90)} 0"/>
       </xacro:set_frame>
     </xacro:macro>
@@ -203,5 +205,5 @@
 			  parent="${prefix}left_finger_spread_link"
 			  mimic_outer_joints="${mimic_outer_joints}">
-      <origin xyz="${inner_x} ${inner_y} ${inner_z}"
+      <origin xyz="${inner_x} 0.0 ${inner_z}"
 	      rpy="${radians(90)} 0.0 0.0"/>
     </xacro:barrett_finger>
@@ -210,5 +212,5 @@
 			  parent="${prefix}right_finger_spread_link"
 			  mimic_outer_joints="${mimic_outer_joints}">
-      <origin xyz="${inner_x} ${inner_y} ${inner_z}"
+      <origin xyz="${inner_x} 0.0 ${inner_z}"
 	      rpy="${radians(90)} 0.0 0.0"/>
     </xacro:barrett_finger>
@@ -217,5 +219,5 @@
 			  parent="${prefix}base_link"
 			  mimic_outer_joints="${mimic_outer_joints}">
-      <origin xyz="${inner_y} ${inner_x} ${base_height + inner_z}"
+      <origin xyz="0.0 ${inner_x} ${base_height + inner_z}"
 	      rpy="${radians(90)} 0.0 ${radians(90)}"/>
     </xacro:barrett_finger>

Commit message: Rename tip_link to tcp_link

File: aist_barrett/urdf/barrett_hand.urdf.xacro (robot description, xacro)
@@ -11,5 +11,5 @@
     <xacro:property name="base_height"		value="0.025"/>
     <xacro:property name="palm_height"		value="0.061"/>
-    <xacro:property name="tip_height"		value="0.156"/>
+    <xacro:property name="tcp_height"		value="0.156"/>
     <xacro:property name="half_tread"		value="0.025"/>
     <xacro:property name="inner_x"		value="0.050"/>
@@ -173,7 +173,7 @@
       <origin xyz="0.0 0.0 ${palm_height}" rpy="0 0 0"/>
     </xacro:set_frame>
-    <xacro:set_frame name="${prefix}tip_link"
+    <xacro:set_frame name="${prefix}tcp_link"
 		     parent="${prefix}base_link">
-      <origin xyz="0.0 0.0 ${tip_height}" rpy="0 ${radians(180)} 0"/>
+      <origin xyz="0.0 0.0 ${tcp_height}" rpy="0 ${radians(180)} 0"/>
     </xacro:set_frame>
     <!-- Spread -->

Commit message: Revert "Rename tip_link to tcp_link"
This reverts commit fdcd73959a6e8cd4dfe0dd2cb6eb6e03d5be8600.

File: aist_barrett/urdf/barrett_hand.urdf.xacro (robot description, xacro)
@@ -11,5 +11,5 @@
     <xacro:property name="base_height"		value="0.025"/>
     <xacro:property name="palm_height"		value="0.061"/>
-    <xacro:property name="tcp_height"		value="0.156"/>
+    <xacro:property name="tip_height"		value="0.156"/>
     <xacro:property name="half_tread"		value="0.025"/>
     <xacro:property name="inner_x"		value="0.050"/>
@@ -173,7 +173,7 @@
       <origin xyz="0.0 0.0 ${palm_height}" rpy="0 0 0"/>
     </xacro:set_frame>
-    <xacro:set_frame name="${prefix}tcp_link"
+    <xacro:set_frame name="${prefix}tip_link"
 		     parent="${prefix}base_link">
-      <origin xyz="0.0 0.0 ${tcp_height}" rpy="0 ${radians(180)} 0"/>
+      <origin xyz="0.0 0.0 ${tip_height}" rpy="0 ${radians(180)} 0"/>
     </xacro:set_frame>
     <!-- Spread -->

Commit message: Make default value of parameter "mimic_joints" false

File: aist_barrett/urdf/barrett_hand.urdf.xacro (robot description, xacro)
@@ -3,5 +3,5 @@
        xmlns:controller="http://playerstage.sourceforge.net/gazebo/xmlschema/#controller">
   <xacro:macro name="barrett_hand"
-	       params="prefix parent_link mimic_outer_joints:=true *origin">
+	       params="prefix parent_link mimic_joints:=false *origin">
     <xacro:macro name="gray_color">
       <material name="">
@@ -26,5 +26,5 @@
     </xacro:macro>
     <xacro:macro name="barrett_finger"
-		 params="fingerprefix parent mimic_outer_joints *origin">
+		 params="fingerprefix parent mimic_joints *origin">
       <joint name="${fingerprefix}joint"
 	     type="revolute">
@@ -70,5 +70,5 @@
 	<child  link="${fingerprefix}outer_link"/>
 	<axis xyz="0 0 1"/>
-	<xacro:if value="${mimic_outer_joints}">
+	<xacro:if value="${mimic_joints}">
 	  <mimic joint="${fingerprefix}joint"
 		 multiplier="${45.0/140.0}" offset="0.0"/>
@@ -194,7 +194,9 @@
       <parent link="${prefix}base_link"/>
       <child  link="${prefix}right_finger_spread_link"/>
-      <axis  xyz="0 0 -1"/>
+      <axis   xyz="0 0 1"/>
+      <xacro:if value="${mimic_joints}">
+	<mimic joint="${prefix}spread_joint" multiplier="1.0" offset="0.0"/>
+      </xacro:if>
       <limit effort="30" velocity="1.5" lower="${radians(180)}" upper="0.0"/>
-      <mimic joint="${prefix}spread_joint" multiplier="-1" offset="0"/>
       <joint_properties damping="100.0" friction="1000.0"/>
       <dynamics damping="1000"/>
@@ -204,5 +206,5 @@
     <xacro:barrett_finger fingerprefix="${prefix}left_finger_"
 			  parent="${prefix}left_finger_spread_link"
-			  mimic_outer_joints="${mimic_outer_joints}">
+			  mimic_joints="${mimic_joints}">
       <origin xyz="${inner_x} 0.0 ${inner_z}"
 	      rpy="${radians(90)} 0.0 0.0"/>
@@ -211,5 +213,5 @@
     <xacro:barrett_finger fingerprefix="${prefix}right_finger_"
 			  parent="${prefix}right_finger_spread_link"
-			  mimic_outer_joints="${mimic_outer_joints}">
+			  mimic_joints="${mimic_joints}">
       <origin xyz="${inner_x} 0.0 ${inner_z}"
 	      rpy="${radians(90)} 0.0 0.0"/>
@@ -218,5 +220,5 @@
     <xacro:barrett_finger fingerprefix="${prefix}middle_finger_"
 			  parent="${prefix}base_link"
-			  mimic_outer_joints="${mimic_outer_joints}">
+			  mimic_joints="${mimic_joints}">
       <origin xyz="0.0 ${inner_x} ${base_height + inner_z}"
 	      rpy="${radians(90)} 0.0 ${radians(90)}"/>

Commit message: Improve transmissions

File: aist_barrett/urdf/barrett_hand.urdf.xacro (robot description, xacro)
@@ -2,4 +2,5 @@
 <robot xmlns:xacro="http://www.ros.org/wiki/xacro"
        xmlns:controller="http://playerstage.sourceforge.net/gazebo/xmlschema/#controller">
+  <xacro:include filename="$(find aist_barrett)/urdf/transmission.urdf.xacro"/>
   <xacro:macro name="barrett_hand"
 	       params="prefix parent_link mimic_joints:=false *origin">
@@ -227,4 +228,5 @@
 		       )/urdf/palm_tactile_sensors.urdf.xacro"/>
     <palm_tactile_sensors/>
+    <xacro:barrett_hand_transmission prefix="${prefix}"/>
   </xacro:macro>
 </robot>

File: aist_barrett/urdf/transmission.urdf.xacro (robot description, xacro)
@@ -1,16 +1,16 @@
 <?xml version="1.0"?>
 <robot xmlns:xacro="http://www.ros.org/wiki/xacro" xmlns:controller="http://playerstage.sourceforge.net/gazebo/xmlschema/#controller">
-  <xacro:macro name="wam_transmission" params="dof hand">
-    <if value="${dof == 4}">
-      <transmission name="trans_q1">
+  <xacro:macro name="barrett_hand_transmission" params="prefix">
+    <xacro:macro name="joint_transmission" params="joint_name">
+      <transmission name="${joint_name}_trans">
 	<type>
 	  transmission_interface/SimpleTransmission
 	</type>
-	<joint name="q1">
+	<joint name="${joint_name}">
 	  <hardwareInterface>
 	    hardware_interface/PositionJointInterface
 	  </hardwareInterface>
 	</joint>
-	<actuator name="q1_motor">
+	<actuator name="${joint_name}_motor">
 	  <hardwareInterface>
 	    hardware_interface/PositionJointInterface
@@ -21,340 +21,13 @@
 	</actuator>
       </transmission>
-      <transmission name="trans_q2">
-	<type>
-	  transmission_interface/SimpleTransmission
-	</type>
-	<joint name="q2">
-	  <hardwareInterface>
-	    hardware_interface/PositionJointInterface
-	  </hardwareInterface>
-	</joint>
-	<actuator name="q2_motor">
-	  <hardwareInterface>
-	    hardware_interface/PositionJointInterface
-	  </hardwareInterface>
-	  <mechanicalReduction>
-	    1
-	  </mechanicalReduction>
-	</actuator>
-      </transmission>
-      <transmission name="trans_q3">
-	<type>
-	  transmission_interface/SimpleTransmission
-	</type>
-	<joint name="q3">
-	  <hardwareInterface>
-	    hardware_interface/PositionJointInterface
-	  </hardwareInterface>
-	</joint>
-	<actuator name="q3_motor">
-	  <hardwareInterface>
-	    hardware_interface/PositionJointInterface
-	  </hardwareInterface>
-	  <mechanicalReduction>
-	    1
-	  </mechanicalReduction>
-	</actuator>
-      </transmission>
-      <transmission name="trans_q4">
-	<type>
-	  transmission_interface/SimpleTransmission
-	</type>
-	<joint name="q4">
-	  <hardwareInterface>
-	    hardware_interface/PositionJointInterface
-	  </hardwareInterface>
-	</joint>
-	<actuator name="q4_motor">
-	  <hardwareInterface>
-	    hardware_interface/PositionJointInterface
-	  </hardwareInterface>
-	  <mechanicalReduction>
-	    1
-	  </mechanicalReduction>
-	</actuator>
-      </transmission>
-    </if>
-    <if value="${dof == 7}">
-      <transmission name="trans_q1">
-	<type>
-	  transmission_interface/SimpleTransmission
-	</type>
-	<joint name="q1">
-	  <hardwareInterface>
-	    hardware_interface/PositionJointInterface
-	  </hardwareInterface>
-	</joint>
-	<actuator name="q1_motor">
-	  <hardwareInterface>
-	    hardware_interface/PositionJointInterface
-	  </hardwareInterface>
-	  <mechanicalReduction>
-	    1
-	  </mechanicalReduction>
-	</actuator>
-      </transmission>
-      <transmission name="trans_q2">
-	<type>
-	  transmission_interface/SimpleTransmission
-	</type>
-	<joint name="q2">
-	  <hardwareInterface>
-	    hardware_interface/PositionJointInterface
-	  </hardwareInterface>
-	</joint>
-	<actuator name="q2_motor">
-	  <hardwareInterface>
-	    hardware_interface/PositionJointInterface
-	  </hardwareInterface>
-	  <mechanicalReduction>
-	    1
-	  </mechanicalReduction>
-	</actuator>
-      </transmission>
-      <transmission name="trans_q3">
-	<type>
-	  transmission_interface/SimpleTransmission
-	</type>
-	<joint name="q3">
-	  <hardwareInterface>
-	    hardware_interface/PositionJointInterface
-	  </hardwareInterface>
-	</joint>
-	<actuator name="q3_motor">
-	  <hardwareInterface>
-	    hardware_interface/PositionJointInterface
-	  </hardwareInterface>
-	  <mechanicalReduction>
-	    1
-	  </mechanicalReduction>
-	</actuator>
-      </transmission>
-      <transmission name="trans_q4">
-	<type>
-	  transmission_interface/SimpleTransmission
-	</type>
-	<joint name="q4">
-	  <hardwareInterface>
-	    hardware_interface/PositionJointInterface
-	  </hardwareInterface>
-	</joint>
-	<actuator name="q4_motor">
-	  <hardwareInterface>
-	    hardware_interface/PositionJointInterface
-	  </hardwareInterface>
-	  <mechanicalReduction>
-	    1
-	  </mechanicalReduction>
-	</actuator>
-      </transmission>
-      <transmission name="trans_q5">
-	<type>
-	  transmission_interface/SimpleTransmission
-	</type>
-	<joint name="q5">
-	  <hardwareInterface>
-	    hardware_interface/PositionJointInterface
-	  </hardwareInterface>
-	</joint>
-	<actuator name="q5_motor">
-	  <hardwareInterface>
-	    hardware_interface/PositionJointInterface
-	  </hardwareInterface>
-	  <mechanicalReduction>
-	    1
-	  </mechanicalReduction>
-	</actuator>
-      </transmission>
-      <transmission name="trans_q6">
-	<type>
-	  transmission_interface/SimpleTransmission
-	</type>
-	<joint name="q6">
-	  <hardwareInterface>
-	    hardware_interface/PositionJointInterface
-	  </hardwareInterface>
-	</joint>
-	<actuator name="q6_motor">
-	  <hardwareInterface>
-	    hardware_interface/PositionJointInterface
-	  </hardwareInterface>
-	  <mechanicalReduction>
-	    1
-	  </mechanicalReduction>
-	</actuator>
-      </transmission>
-      <transmission name="trans_q7">
-	<type>
-	  transmission_interface/SimpleTransmission
-	</type>
-	<joint name="q7">
-	  <hardwareInterface>
-	    hardware_interface/PositionJointInterface
-	  </hardwareInterface>
-	</joint>
-	<actuator name="q7_motor">
-	  <hardwareInterface>
-	    hardware_interface/PositionJointInterface
-	  </hardwareInterface>
-	  <mechanicalReduction>
-	    1
-	  </mechanicalReduction>
-	</actuator>
-      </transmission>
-    </if>
-    <if value="${hand == 1}">
-      <transmission name="trans_bhand_j11_joint">
-	<type>
-	  transmission_interface/SimpleTransmission
-	</type>
-	<joint name="bhand_j11_joint">
-	  <hardwareInterface>
-	    hardware_interface/PositionJointInterface
-	  </hardwareInterface>
-	</joint>
-	<actuator name="bhand_j11_joint_motor">
-	  <hardwareInterface>
-	    hardware_interface/PositionJointInterface
-	  </hardwareInterface>
-	  <mechanicalReduction>
-	    1
-	  </mechanicalReduction>
-	</actuator>
-      </transmission>
-      <transmission name="trans_bhand_j21_joint">
-	<type>
-	  transmission_interface/SimpleTransmission
-	</type>
-	<joint name="bhand_j21_joint">
-	  <hardwareInterface>
-	    hardware_interface/PositionJointInterface
-	  </hardwareInterface>
-	</joint>
-	<actuator name="bhand_j21_joint_motor">
-	  <hardwareInterface>
-	    hardware_interface/PositionJointInterface
-	  </hardwareInterface>
-	  <mechanicalReduction>
-	    1
-	  </mechanicalReduction>
-	</actuator>
-      </transmission>
-      <transmission name="trans_bhand_j12_joint">
-	<type>
-	  transmission_interface/SimpleTransmission
-	</type>
-	<joint name="bhand_j12_joint">
-	  <hardwareInterface>
-	    hardware_interface/PositionJointInterface
-	  </hardwareInterface>
-	</joint>
-	<actuator name="bhand_j12_joint_motor">
-	  <hardwareInterface>
-	    hardware_interface/PositionJointInterface
-	  </hardwareInterface>
-	  <mechanicalReduction>
-	    1
-	  </mechanicalReduction>
-	</actuator>
-      </transmission>
-      <transmission name="trans_bhand_j22_joint">
-	<type>
-	  transmission_interface/SimpleTransmission
-	</type>
-	<joint name="bhand_j22_joint">
-	  <hardwareInterface>
-	    hardware_interface/PositionJointInterface
-	  </hardwareInterface>
-	</joint>
-	<actuator name="bhand_j22_joint_motor">
-	  <hardwareInterface>
-	    hardware_interface/PositionJointInterface
-	  </hardwareInterface>
-	  <mechanicalReduction>
-	    1
-	  </mechanicalReduction>
-	</actuator>
-      </transmission>
-      <transmission name="trans_bhand_j32_joint">
-	<type>
-	  transmission_interface/SimpleTransmission
-	</type>
-	<joint name="bhand_j32_joint">
-	  <hardwareInterface>
-	    hardware_interface/PositionJointInterface
-	  </hardwareInterface>
-	</joint>
-	<actuator name="bhand_j32_joint_motor">
-	  <hardwareInterface>
-	    hardware_interface/PositionJointInterface
-	  </hardwareInterface>
-	  <mechanicalReduction>
-	    1
-	  </mechanicalReduction>
-	</actuator>
-      </transmission>
-      <transmission name="trans_bhand_j13_joint">
-	<type>
-	  transmission_interface/SimpleTransmission
-	</type>
-	<joint name="bhand_j13_joint">
-	  <hardwareInterface>
-	    hardware_interface/PositionJointInterface
-	  </hardwareInterface>
-	</joint>
-	<actuator name="bhand_j13_joint_motor">
-	  <hardwareInterface>
-	    hardware_interface/PositionJointInterface
-	  </hardwareInterface>
-	  <mechanicalReduction>
-	    1
-	  </mechanicalReduction>
-	</actuator>
-      </transmission>
-      <transmission name="trans_bhand_j23_joint">
-	<type>
-	  transmission_interface/SimpleTransmission
-	</type>
-	<joint name="bhand_j23_joint">
-	  <hardwareInterface>
-	    hardware_interface/PositionJointInterface
-	  </hardwareInterface>
-	</joint>
-	<actuator name="bhand_j23_joint_motor">
-	  <hardwareInterface>
-	    hardware_interface/PositionJointInterface
-	  </hardwareInterface>
-	  <mechanicalReduction>
-	    1
-	  </mechanicalReduction>
-	</actuator>
-      </transmission>
-      <transmission name="trans_bhand_j33_joint">
-	<type>
-	  transmission_interface/SimpleTransmission
-	</type>
-	<joint name="bhand_j33_joint">
-	  <hardwareInterface>
-	    hardware_interface/PositionJointInterface
-	  </hardwareInterface>
-	</joint>
-	<actuator name="bhand_j33_joint_motor">
-	  <hardwareInterface>
-	    hardware_interface/PositionJointInterface
-	  </hardwareInterface>
-	  <mechanicalReduction>
-	    1
-	  </mechanicalReduction>
-	</actuator>
-      </transmission>
-    </if>
-    <gazebo>
-      <plugin name="gazebo_ros_control" filename="libgazebo_ros_control.so">
-	<robotNamespace>
-	  /
-	</robotNamespace>
-      </plugin>
-    </gazebo>
+    </xacro:macro>
+    <xacro:joint_transmission joint_name="${prefix}left_finger_joint"/>
+    <xacro:joint_transmission joint_name="${prefix}right_finger_joint"/>
+    <xacro:joint_transmission joint_name="${prefix}middle_finger_joint"/>
+    <xacro:joint_transmission joint_name="${prefix}spread_joint"/>
+    <xacro:joint_transmission joint_name="${prefix}left_finger_outer_joint"/>
+    <xacro:joint_transmission joint_name="${prefix}right_finger_outer_joint"/>
+    <xacro:joint_transmission joint_name="${prefix}middle_finger_outer_joint"/>
+    <xacro:joint_transmission joint_name="${prefix}right_spread_joint"/>
   </xacro:macro>
 </robot>
